File: PCB activity/PCB activity.kicad_sch (KiCad schematic)
At the start: 13 parts, among them J1 Conn_01x08, J2 Conn_01x08

Commit message: added mikroBUS footprint
Parts:
- D1, D2, D3, D4, D5: footprint (none) -> LED_SMD:LED_0805_2012Metric
- R1, R2, R3, R4, R5: footprint (none) -> Resistor_SMD:R_0805_2012Metric
Connections:
- net GND: now also J1.8 (Pin_8), U1.4 (GND)
- net +3.3V: now reaches D1.2 (A)
- net +3.3V: now also J1.7 (Pin_7), U1.1 (VDDD), U1.7 (SERMODE), U1.8 (VDDA)
- net CS: now reaches D3.2 (A)
- net CS: now also J1.3 (Pin_3), U1.3 (SCLK)
- net SCK: now reaches D2.2 (A)
- net SCK: now also J1.4 (Pin_4), U1.2 (CE)
- net MOSI: now reaches D4.2 (A)
- net MOSI: now also J1.6 (Pin_6), U1.6 (SDI)
- net MISO: now reaches D5.2 (A)
- net MISO: now also J1.5 (Pin_5), U1.5 (SDO)
- no-connect marks 0 -> 10
Changed lines of the file:
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@@
 (kicad_sch (version 20230121) (generator eeschema)
   (paper "A4")
+  (no_connect (at 156.21 64.77))
+  (no_connect (at 156.21 62.23))
+  (no_connect (at 156.21 57.15))
+  (no_connect (at 156.21 67.31))
+  (no_connect (at 156.21 54.61))
+  (no_connect (at 156.21 59.69))
+  (no_connect (at 156.21 52.07))
+  (no_connect (at 76.2 50.8))
+  (no_connect (at 76.2 48.26))
+  (no_connect (at 156.21 49.53))
+  (wire (pts (xy 91.44 110.49) (xy 99.06 110.49))
+    (stroke (width 0) (type default))
+  )
+  (wire (pts (xy 58.42 118.11) (xy 66.04 118.11))
+    (stroke (width 0) (type default))
+  )
   (wire (pts (xy 168.91 104.14) (xy 168.91 109.22))
     (stroke (width 0) (type default))
   )
+  (wire (pts (xy 168.91 90.17) (xy 168.91 96.52))
+    (stroke (width 0) (type default))
+  )
+  (wire (pts (xy 68.58 53.34) (xy 76.2 53.34))
+    (stroke (width 0) (type default))
+  )
+  (wire (pts (xy 68.58 58.42) (xy 76.2 58.42))
+    (stroke (width 0) (type default))
+  )
+  (wire (pts (xy 68.58 63.5) (xy 76.2 63.5))
+    (stroke (width 0) (type default))
+  )
+  (wire (pts (xy 68.58 60.96) (xy 76.2 60.96))
+    (stroke (width 0) (type default))
+  )
+  (wire (pts (xy 68.58 55.88) (xy 76.2 55.88))
+    (stroke (width 0) (type default))
+  )
   (wire (pts (xy 146.05 116.84) (xy 146.05 125.73))
     (stroke (width 0) (type default))
   )
+  (wire (pts (xy 134.62 90.17) (xy 134.62 96.52))
+    (stroke (width 0) (type default))
+  )
   (wire (pts (xy 157.48 104.14) (xy 157.48 109.22))
     (stroke (width 0) (type default))
@@
     (stroke (width 0) (type default))
   )
+  (wire (pts (xy 91.44 114.3) (xy 99.06 114.3))
+    (stroke (width 0) (type default))
+  )
+  (wire (pts (xy 58.42 110.49) (xy 66.04 110.49))
+    (stroke (width 0) (type default))
+  )
+  (wire (pts (xy 157.48 90.17) (xy 157.48 96.52))
+    (stroke (width 0) (type default))
+  )
+  (wire (pts (xy 68.58 66.04) (xy 76.2 66.04))
+    (stroke (width 0) (type default))
+  )
+  (wire (pts (xy 123.19 90.17) (xy 123.19 96.52))
+    (stroke (width 0) (type default))
+  )
+  (wire (pts (xy 58.42 106.68) (xy 66.04 106.68))
+    (stroke (width 0) (type default))
+  )
   (wire (pts (xy 168.91 116.84) (xy 168.91 125.73))
     (stroke (width 0) (type default))
@@
     (stroke (width 0) (type default))
   )
+  (wire (pts (xy 91.44 106.68) (xy 99.06 106.68))
+    (stroke (width 0) (type default))
+  )
+  (wire (pts (xy 91.44 118.11) (xy 99.06 118.11))
+    (stroke (width 0) (type default))
+  )
   (wire (pts (xy 123.19 116.84) (xy 123.19 125.73))
     (stroke (width 0) (type default))
   )
+  (wire (pts (xy 146.05 90.17) (xy 146.05 96.52))
+    (stroke (width 0) (type default))
+  )
   (wire (pts (xy 146.05 104.14) (xy 146.05 109.22))
     (stroke (width 0) (type default))
   )
+  (wire (pts (xy 58.42 114.3) (xy 66.04 114.3))
+    (stroke (width 0) (type default))
+  )
   (wire (pts (xy 157.48 116.84) (xy 157.48 125.73))
     (stroke (width 0) (type default))
@@
     (effects (font (size 1.27 1.27)) (justify left bottom))
   )
+  (label "SCK" (at 58.42 110.49 0) (fields_autoplaced)
+    (effects (font (size 1.27 1.27)) (justify left bottom))
+  )
+  (label "CS" (at 58.42 114.3 0) (fields_autoplaced)
+    (effects (font (size 1.27 1.27)) (justify left bottom))
+  )
+  (label "+3.3V" (at 99.06 110.49 180) (fields_autoplaced)
+    (effects (font (size 1.27 1.27)) (justify right bottom))
+  )
+  (label "SCK" (at 68.58 55.88 0) (fields_autoplaced)
+    (effects (font (size 1.27 1.27)) (justify left bottom))
+  )
+  (label "GND" (at 68.58 66.04 0) (fields_autoplaced)
+    (effects (font (size 1.27 1.27)) (justify left bottom))
+  )
+  (label "MOSI" (at 68.58 60.96 0) (fields_autoplaced)
+    (effects (font (size 1.27 1.27)) (justify left bottom))
+  )
+  (label "MOSI" (at 157.48 90.17 0) (fields_autoplaced)
+    (effects (font (size 1.27 1.27)) (justify left bottom))
+  )
+  (label "+3.3V" (at 99.06 106.68 180) (fields_autoplaced)
+    (effects (font (size 1.27 1.27)) (justify right bottom))
+  )
+  (label "MOSI" (at 99.06 114.3 180) (fields_autoplaced)
+    (effects (font (size 1.27 1.27)) (justify right bottom))
+  )
+  (label "MISO" (at 168.91 90.17 0) (fields_autoplaced)
+    (effects (font (size 1.27 1.27)) (justify left bottom))
+  )
+  (label "MISO" (at 68.58 58.42 0) (fields_autoplaced)
+    (effects (font (size 1.27 1.27)) (justify left bottom))
+  )
+  (label "GND" (at 58.42 118.11 0) (fields_autoplaced)
+    (effects (font (size 1.27 1.27)) (justify left bottom))
+  )
+  (label "SCK" (at 134.62 90.17 0) (fields_autoplaced)
+    (effects (font (size 1.27 1.27)) (justify left bottom))
+  )
+  (label "+3.3V" (at 58.42 106.68 0) (fields_autoplaced)
+    (effects (font (size 1.27 1.27)) (justify left bottom))
+  )
+  (label "MISO" (at 99.06 118.11 180) (fields_autoplaced)
+    (effects (font (size 1.27 1.27)) (justify right bottom))
+  )
+  (label "CS" (at 68.58 53.34 0) (fields_autoplaced)
+    (effects (font (size 1.27 1.27)) (justify left bottom))
+  )
+  (label "+3.3V" (at 123.19 90.17 0) (fields_autoplaced)
+    (effects (font (size 1.27 1.27)) (justify left bottom))
+  )
+  (label "+3.3V" (at 68.58 63.5 0) (fields_autoplaced)
+    (effects (font (size 1.27 1.27)) (justify left bottom))
+  )
+  (label "CS" (at 146.05 90.17 0) (fields_autoplaced)
+    (effects (font (size 1.27 1.27)) (justify left bottom))
+  )
   (symbol (lib_id "Device:R") (at 146.05 113.03 0) (unit 1)
     (in_bom yes) (on_board yes) (dnp no) (fields_autoplaced)
@@
       (effects (font (size 1.27 1.27)) (justify left))
     )
-    (property "Footprint" "" (at 144.272 113.03 90)
+    (property "Footprint" "Resistor_SMD:R_0805_2012Metric" (at 144.272 113.03 90)
       (effects (font (size 1.27 1.27)) hide)
     )
@@
       (effects (font (size 1.27 1.27)) (justify left))
     )
-    (property "Footprint" "" (at 155.702 113.03 90)
+    (property "Footprint" "Resistor_SMD:R_0805_2012Metric" (at 155.702 113.03 90)
       (effects (font (size 1.27 1.27)) hide)
     )
@@
       (effects (font (size 1.27 1.27)) (justify left))
     )
-    (property "Footprint" "" (at 132.842 113.03 90)
+    (property "Footprint" "Resistor_SMD:R_0805_2012Metric" (at 132.842 113.03 90)
       (effects (font (size 1.27 1.27)) hide)
     )
@@
       (effects (font (size 1.27 1.27)) (justify right))
     )
-    (property "Footprint" "" (at 123.19 100.33 0)
+    (property "Footprint" "LED_SMD:LED_0805_2012Metric" (at 123.19 100.33 0)
       (effects (font (size 1.27 1.27)) hide)
     )
@@
       (effects (font (size 1.27 1.27)) (justify left))
     )
-    (property "Footprint" "" (at 167.132 113.03 90)
+    (property "Footprint" "Resistor_SMD:R_0805_2012Metric" (at 167.132 113.03 90)
       (effects (font (size 1.27 1.27)) hide)
     )
@@
       (effects (font (size 1.27 1.27)) (justify left))
     )
-    (property "Footprint" "" (at 121.412 113.03 90)
+    (property "Footprint" "Resistor_SMD:R_0805_2012Metric" (at 121.412 113.03 90)
       (effects (font (size 1.27 1.27)) hide)
     )
@@
       (effects (font (size 1.27 1.27)) (justify right))
     )
-    (property "Footprint" "" (at 146.05 100.33 0)
+    (property "Footprint" "LED_SMD:LED_0805_2012Metric" (at 146.05 100.33 0)
       (effects (font (size 1.27 1.27)) hide)
     )
@@
       (effects (font (size 1.27 1.27)) (justify right))
     )
-    (property "Footprint" "" (at 134.62 100.33 0)
+    (property "Footprint" "LED_SMD:LED_0805_2012Metric" (at 134.62 100.33 0)
       (effects (font (size 1.27 1.27)) hide)
     )
@@
       (effects (font (size 1.27 1.27)) (justify right))
     )
-    (property "Footprint" "" (at 157.48 100.33 0)
+    (property "Footprint" "LED_SMD:LED_0805_2012Metric" (at 157.48 100.33 0)
       (effects (font (size 1.27 1.27)) hide)
     )
@@
       (effects (font (size 1.27 1.27)) (justify right))
     )
-    (property "Footprint" "" (at 168.91 100.33 0)
-      (effects (font (size 1.27 1.27)) hide)
-    )
+    (property "Footprint" "LED_SMD:LED_0805_2012Metric" (at 168.91 100.33 0)
+      (effects (font (size 1.27 1.27)) hide)
+    )

Commit message: added DS1722 footprint
Parts:
- U1: footprint (none) -> DS1722:DS1722
Changed lines of the file:
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@@
       (effects (font (size 1.27 1.27)))
     )
-    (property "Footprint" "" (at 78.74 113.03 0)
-      (effects (font (size 1.27 1.27)) hide)
+    (property "Footprint" "DS1722:DS1722" (at 78.74 113.03 0)
+      (effects (font (size 1.27 1.27)))
     )
     (property "Datasheet" "" (at 78.74 113.03 0)
